Commit message: fixed now removed config reference

File: src/apollo_description/urdf/sensors/camera_bracket.urdf.xacro (robot description, xacro)
@@ -14,5 +14,5 @@
     <visual>
       <geometry>
-       <mesh filename="package://apollo_description/meshes/camera_bracket.dae" scale="1 1 1" />
+       <mesh filename="package://apollo_description/meshes/turtlebot/camera_bracket.dae" scale="1 1 1" />
       </geometry>
     </visual>

File: src/apollo_description/urdf/sensors/oakd.urdf.xacro (robot description, xacro)
@@ -22,5 +22,5 @@
     <visual>
       <geometry>
-        <mesh filename="package://apollo_description/meshes/${name}_${model}.dae" scale="1 1 1" />
+        <mesh filename="package://apollo_description/meshes/turtlebot/${name}_${model}.dae" scale="1 1 1" />
       </geometry>
     </visual>

File: src/apollo_description/urdf/sensors/rplidar.urdf.xacro (robot description, xacro)
@@ -18,5 +18,5 @@
     <visual>
       <geometry>
-        <mesh filename="package://apollo_description/meshes/rplidar.dae" scale="1 1 1" />
+        <mesh filename="package://apollo_description/meshes/turtlebot/rplidar.dae" scale="1 1 1" />
       </geometry>
     </visual>

File: src/apollo_description/urdf/standard/apollo.urdf.xacro (robot description, xacro)
@@ -43,10 +43,10 @@
       <origin xyz="0 0 0" rpy="${pi/2} 0 ${pi/2}"/>
       <geometry>
-        <mesh filename="package://apollo_description/meshes/shell.dae" scale="1 1 1" />
+        <mesh filename="package://apollo_description/meshes/turtlebot/shell.dae" scale="1 1 1" />
       </geometry>
     </visual>
     <collision name="shell_collision">
       <geometry>
-        <mesh filename="package://apollo_description/meshes/shell_collision.dae" scale="1 1 1" />
+        <mesh filename="package://apollo_description/meshes/turtlebot/shell_collision.dae" scale="1 1 1" />
       </geometry>
     </collision>

File: src/apollo_description/urdf/standard/tower_sensor_plate.urdf.xacro (robot description, xacro)
@@ -14,5 +14,5 @@
     <visual>
       <geometry>
-       <mesh filename="package://apollo_description/meshes/tower_sensor_plate.dae" scale="1 1 1" />
+       <mesh filename="package://apollo_description/meshes/turtlebot/tower_sensor_plate.dae" scale="1 1 1" />
       </geometry>
     </visual>

File: src/apollo_description/urdf/standard/tower_standoff.urdf.xacro (robot description, xacro)
@@ -15,5 +15,5 @@
       <origin rpy="0 ${pi/2} 0"/>
       <geometry>
-       <mesh filename="package://apollo_description/meshes/tower_standoff.dae" scale="1 1 1" />
+       <mesh filename="package://apollo_description/meshes/turtlebot/tower_standoff.dae" scale="1 1 1" />
       </geometry>
     </visual>

File: src/apollo_description/urdf/standard/weight_block.urdf.xacro (robot description, xacro)
@@ -14,5 +14,5 @@
     <visual>
       <geometry>
-       <mesh filename="package://apollo_description/meshes/weight_block.dae" scale="1 1 1" />
+       <mesh filename="package://apollo_description/meshes/turtlebot/weight_block.dae" scale="1 1 1" />
       </geometry>
     </visual>
