Commit message: removed some unnecessary details

File: src/apollo_description/urdf/apollo.imu.xacro (robot description, xacro)
@@ -2,4 +2,5 @@
 <robot xmlns:xacro="http://www.ros.org/wiki/xacro">
     <xacro:macro name="imu_sensor" params="parent prefix *origin">
+        <!-- Fixed joint to parent (chassis) -->
         <joint name="${prefix}_imu_joint" type="fixed">
             <xacro:insert_block name="origin" />
@@ -7,11 +8,6 @@
             <child link="${prefix}_imu_link" />
         </joint>
+        <!-- red box visual -->
         <link name="${prefix}_imu_link">
-            <inertial>
-                <mass value="0.1" />
-                <origin xyz="0 0 0" rpy="0 0 0" />
-                <inertia ixx="0.000166667" ixy="0" ixz="0" iyy="0.000166667" iyz="0"
-                    izz="0.000166667" />
-            </inertial>
             <visual>
                 <geometry>
@@ -23,13 +19,11 @@
             </visual>
         </link>
+        <!-- IMU sensor plugin -->
         <gazebo reference="${prefix}_imu_link">
             <sensor name="${prefix}_imu" type="imu">
                 <always_on>true</always_on>
                 <update_rate>100</update_rate>
-                <visualize>true</visualize>
                 <topic>/imu</topic>
-                <plugin filename="libgz-sim-imu-system.so" name="gz::sim::systems::Imu">
-                    <initial_orientation_as_reference>false</initial_orientation_as_reference>
-                </plugin>
+                <plugin filename="libgz-sim-imu-system.so" name="gz::sim::systems::Imu"/>
             </sensor>
         </gazebo>

File: src/apollo_description/urdf/apollo.urdf.xacro (robot description, xacro)
@@ -4,5 +4,5 @@
   <xacro:include filename="apollo.imu.xacro"/>
   <xacro:imu_sensor prefix="apollo" parent="chassis">
-    <origin xyz="0 0 0" rpy="0 0 0"/>
+    <origin xyz="0 0 0.1" rpy="0 0 0"/>
   </xacro:imu_sensor>
 </robot>
