Commit message: added imu sim

File: src/apollo_description/urdf/apollo.urdf.xacro (robot description, xacro)
@@ -2,3 +2,7 @@
 <robot name="apollo" xmlns:xacro="http://ros.org/wiki/xacro">
   <xacro:include filename="apollo.drive.urdf.xacro" />
+  <xacro:include filename="apollo.imu.xacro"/>
+  <xacro:imu_sensor prefix="apollo" parent="chassis">
+    <origin xyz="0 0 0" rpy="0 0 0"/>
+  </xacro:imu_sensor>
 </robot>

Commit message: added gps sim but it doesnt work

File: src/apollo_description/urdf/apollo.urdf.xacro (robot description, xacro)
@@ -3,6 +3,10 @@
   <xacro:include filename="apollo.drive.urdf.xacro" />
   <xacro:include filename="apollo.imu.xacro"/>
+  <xacro:include filename="apollo.gps.xacro"/>
   <xacro:imu_sensor prefix="apollo" parent="chassis">
     <origin xyz="0 0 0.1" rpy="0 0 0"/>
   </xacro:imu_sensor>
+  <xacro:gps_sensor prefix="apollo" parent="chassis">
+    <origin xyz="0 0.1 0.1" rpy="0 0 0"/>
+  </xacro:gps_sensor>
 </robot>

Commit message: added zed sim

File: src/apollo_description/urdf/apollo.urdf.xacro (robot description, xacro)
@@ -1,3 +1,3 @@
-<?xml version="1.0" ?>
+<?xml version="1.0"?>
 <robot name="apollo" xmlns:xacro="http://ros.org/wiki/xacro">
   <xacro:include filename="apollo.drive.urdf.xacro" />
@@ -5,11 +5,15 @@
   <xacro:apollo_ros2_control name="apollo_drive_control" prefix="apollo" use_mock_hardware='true'>
   </xacro:apollo_ros2_control>
-  <xacro:include filename="apollo.imu.xacro"/>
-  <xacro:include filename="apollo.gps.xacro"/>
+  <xacro:include filename="apollo.imu.xacro" />
+  <xacro:include filename="apollo.gps.xacro" />
+  <xacro:include filename="apollo.zed2.urdf.xacro" />
   <xacro:imu_sensor prefix="apollo" parent="chassis">
-    <origin xyz="0 0 0.1" rpy="0 0 0"/>
+    <origin xyz="0 0 0.1" rpy="0 0 0" />
   </xacro:imu_sensor>
   <xacro:gps_sensor prefix="apollo" parent="chassis">
-    <origin xyz="0 0.1 0.1" rpy="0 0 0"/>
+    <origin xyz="0 0.1 0.1" rpy="0 0 0" />
   </xacro:gps_sensor>
+  <xacro:zed2_camera name="zed2" parent_link="chassis" topic_prefix="apollo/zed2">
+    <origin xyz="0.2 0 0.1" rpy="0 0 0" />
+  </xacro:zed2_camera>
 </robot>
